Commit message: Initial setup completed

File: slam_project/urdf/udacity_bot.xacro (robot description, xacro)
@@ -104,8 +104,8 @@
 	<joint name="camera_joint" type="fixed" >
 		<parent link="chassis"/>
-		<child link="camera"/>
+		<child link="camera_link"/>
 		<origin xyz="0.2 0 0" rpy="0 0 0"/>
 	</joint>
-	<link name='camera'>
+	<link name='camera_link'>
 		<inertial>
 			<mass value="0.1"/>
@@ -130,4 +130,11 @@
 		</visual>
 	</link>
+	<link name='camera_rgbd_frame'>
+	</link>
+	<joint name="camera_rgbd_joint" type="fixed" >
+		<parent link="camera_link"/>
+		<child link="camera_rgbd_frame"/>
+		<origin xyz="0 0 0" rpy="0 0 0"/>
+	</joint>
 	<joint name="hokuyo_joint" type="fixed" >
 		<parent link="chassis"/>

Commit message: Correct kinect camera orientation

File: slam_project/urdf/udacity_bot.xacro (robot description, xacro)
@@ -110,5 +110,5 @@
 		<inertial>
 			<mass value="0.1"/>
-			<origin xyz="0.0 0 0" rpy="0 0 0"/>
+			<origin xyz="0.0 0 0" rpy="0.0 0 0"/>
 			<inertia
 			  ixx="1e-6" ixy="0" ixz="0"
@@ -130,10 +130,9 @@
 		</visual>
 	</link>
-	<link name='camera_rgbd_frame'>
-	</link>
+	<link name='camera_rgbd_frame'></link>
 	<joint name="camera_rgbd_joint" type="fixed" >
 		<parent link="camera_link"/>
 		<child link="camera_rgbd_frame"/>
-		<origin xyz="0 0 0" rpy="0 0 0"/>
+		<origin xyz="0 0 0" rpy="-1.57 0 -1.57"/>
 	</joint>
 	<joint name="hokuyo_joint" type="fixed" >
