Commit message: Update model

File: slam_project/urdf/robokoko_scratch.xacro (robot description, xacro)
@@ -2,23 +2,7 @@
 <robot name="robokoko_bot" xmlns:xacro="http://www.ros.org/wiki/xacro">
   <xacro:include filename="$(find slam_project)/urdf/robokoko_scratch.gazebo" />
-	<gazebo reference="left_wheel_link">
-		<material>Gazebo/Yellow</material>
-	</gazebo>
-	<gazebo reference="right_wheel_link">
-		<material>Gazebo/Yellow</material>
-	</gazebo>
-	<gazebo reference="chassis_link">
-		<material>Gazebo/Black</material>
-	</gazebo>
-	<gazebo reference="body_link">
-		<material>Gazebo/Orange</material>
-	</gazebo>
-	<gazebo reference="camera_link">
-		<material>Gazebo/Orange</material>
-	</gazebo>
-	<gazebo reference="front_caster_link">
-		<material>Gazebo/Orange</material>
-	</gazebo>
+	<!-- Link robot footprint -->
   <link name="robot_footprint"/>
+	<!-- Link chassis -->
   <link name="chassis_link">
 		<visual>
@@ -39,4 +23,5 @@
     </inertial>
   </link>
+	<!-- Link Front Caster -->
 	<link name='front_caster_link'>
 		<visual>
@@ -53,10 +38,32 @@
 			<mass value=".250"/>
 			<inertia
-			  ixx="0." ixy="0" ixz="0"
-			  iyy="0." iyz="0"
-			  izz="0."
-			/>
-		</inertial>
-	</link>
+			  ixx="0.000703125" ixy="0" ixz="0"
+			  iyy="0.000703125" iyz="0"
+			  izz="0.000703125"
+			/>
+		</inertial>
+	</link>
+	<!-- Link Back Caster -->
+	<link name='back_caster_link'>
+		<visual>
+		  <geometry>
+				<sphere radius="0.075"/>
+		  </geometry>
+		</visual>
+		<collision name='back_caster_collision'>
+		  <geometry>
+				<sphere radius="0.075"/>
+		  </geometry>
+		</collision>
+		<inertial>
+			<mass value=".250"/>
+			<inertia
+			  ixx="0.000703125" ixy="0" ixz="0"
+			  iyy="0.000703125" iyz="0"
+			  izz="0.000703125"
+			/>
+		</inertial>
+	</link>
+	<!-- Link Left Wheel -->
 	<link name='left_wheel_link'>
 		<visual>
@@ -82,4 +89,5 @@
 		</inertial>
 	</link>
+	<!-- Link Right Wheel -->
 	<link name='right_wheel_link'>
 		<visual>
@@ -104,4 +112,5 @@
 		</inertial>
 	</link>
+	<!-- Link Body -->
 	<link name='body_link'>
 		<visual>
@@ -112,5 +121,5 @@
 		<collision name='body_collision'>
 		  <geometry>
-				<cylinder length="0.8" radius="0.1"/>
+				<cylinder length="0.65" radius="0.1"/>
 		  </geometry>
 		</collision>
@@ -124,4 +133,5 @@
 		</inertial>
 	</link>
+	<!-- Link Camera -->
 	<link name='camera_link'>
 		<visual>
@@ -144,5 +154,8 @@
 		</inertial>
 	</link>
+	<!-- Link RGB-D  -->
 	<link name='camera_rgbd_frame'></link>
+	<link name='imu_link'></link>
+	<!-- Link Lidar  -->
 	<link name='hokuyo'>
 		<visual>
@@ -167,4 +180,5 @@
 		</inertial>
 	</link>
+	<!-- Joint Robot footprint  -->
   <joint name="robot_footprint_joint" type="fixed">
 	  <origin xyz="0 0 0.15" rpy="0 0 0" />
@@ -172,21 +186,31 @@
     <child link="chassis_link"/>
   </joint>
+	<!-- Joint left wheel  -->
 	<joint name="left_wheel_joint" type="continuous" >
-		<origin xyz="-0.1 0.35 0" rpy="0 0 0"/>
+		<origin xyz="0 0.35 0" rpy="0 0 0"/>
 		<axis xyz="0 1 0" />
 		<parent link="chassis_link"/>
 		<child link="left_wheel_link"/>
 	</joint>
+	<!-- Joint right wheel  -->
 	<joint name="right_wheel_joint" type="continuous" >
-    <origin xyz="-0.1 -0.35 0" rpy="0 0 0"/>
+    <origin xyz="0 -0.35 0" rpy="0 0 0"/>
 		<axis xyz="0 1 0" />
 		<parent link="chassis_link"/>
 		<child link="right_wheel_link"/>
 	</joint>
+	<!-- Joint front caster  -->
 	<joint name="front_caster_joint" type="fixed" >
-		<origin xyz="0.15 0 -0.075" rpy="0 0 0"/>
+		<origin xyz="0.22 0 -0.075" rpy="0 0 0"/>
 		<parent link="chassis_link"/>
 		<child link="front_caster_link"/>
 	</joint>
+	<!-- Joint back caster  -->
+	<joint name="back_caster_joint" type="fixed" >
+		<origin xyz="-0.22 0 -0.075" rpy="0 0 0"/>
+		<parent link="chassis_link"/>
+		<child link="back_caster_link"/>
+	</joint>
+	<!-- Joint body  -->
 	<joint name="body_joint" type="fixed" >
 		<origin xyz="0 0 0.45" rpy="0 0 0"/>
@@ -194,4 +218,5 @@
 		<child link="body_link"/>
 	</joint>
+	<!-- Joint lidar  -->
 	<joint name="lidar_joint" type="fixed" >
     <origin xyz="0 0 0.435" rpy="0 0 0"/>
@@ -199,4 +224,5 @@
 		<child link="hokuyo"/>
 	</joint>
+	<!-- Joint camera  -->
 	<joint name="camera_joint" type="fixed" >
     <origin xyz="0.11 0 0.2" rpy="0 0 0"/>
@@ -204,4 +230,5 @@
 		<child link="camera_link"/>
 	</joint>
+	<!-- Joint camera rgbd  -->
 	<joint name="camera_rgbd_joint" type="fixed" >
 		<parent link="camera_link"/>
@@ -209,3 +236,9 @@
 		<origin xyz="0 0 0" rpy="-1.57 0 -1.57"/>
 	</joint>
+	<!-- Joint Imu  -->
+	<joint name="imu_joint" type="fixed" >
+		<parent link="body_link"/>
+		<child link="imu_link"/>
+		<origin xyz="0 0 0" rpy="0 0 0"/>
+	</joint>
 </robot>

Commit message: Project beta 1

File: slam_project/urdf/robokoko_scratch.xacro (robot description, xacro)
@@ -8,17 +8,17 @@
 		<visual>
       <geometry>
-      	<cylinder length="0.1" radius="0.3"/>
+      	<cylinder length="0.05" radius="0.15"/>
       </geometry>
     </visual>
     <collision name="collision">
       <geometry>
-        <cylinder length="0.1" radius="0.3"/>
+      	<cylinder length="0.05" radius="0.15"/>
       </geometry>
     </collision>
     <inertial>
-      <mass value="10.0"/>
-      <inertia 	ixx="0.35" ixy="0" ixz="0"
-								iyy="0.35" iyz="0"
-						 		izz="0.675"/>
+      <mass value="2.0"/>
+      <inertia 	ixx="0.011666666666666665" ixy="0" ixz="0"
+								iyy="0.011666666666666665" iyz="0"
+						 		izz="0.0225"/>
     </inertial>
   </link>
@@ -27,18 +27,18 @@
 		<visual>
 		  <geometry>
-				<sphere radius="0.075"/>
+				<sphere radius="0.0375"/>
 		  </geometry>
 		</visual>
 		<collision name='front_caster_collision'>
 		  <geometry>
-				<sphere radius="0.075"/>
-		  </geometry>
-		</collision>
-		<inertial>
-			<mass value=".250"/>
-			<inertia
-			  ixx="0.000703125" ixy="0" ixz="0"
-			  iyy="0.000703125" iyz="0"
-			  izz="0.000703125"
+				<sphere radius="0.0375"/>
+		  </geometry>
+		</collision>
+		<inertial>
+			<mass value=".100"/>
+			<inertia
+			  ixx="5.6250000000000005e-05" ixy="0" ixz="0"
+			  iyy="5.6250000000000005e-05" iyz="0"
+			  izz="5.6250000000000005e-05"
 			/>
 		</inertial>
@@ -48,18 +48,18 @@
 		<visual>
 		  <geometry>
-				<sphere radius="0.075"/>
+				<sphere radius="0.0375"/>
 		  </geometry>
 		</visual>
 		<collision name='back_caster_collision'>
 		  <geometry>
-				<sphere radius="0.075"/>
-		  </geometry>
-		</collision>
-		<inertial>
-			<mass value=".250"/>
-			<inertia
-			  ixx="0.000703125" ixy="0" ixz="0"
-			  iyy="0.000703125" iyz="0"
-			  izz="0.000703125"
+				<sphere radius="0.0375"/>
+		  </geometry>
+		</collision>
+		<inertial>
+			<mass value=".100"/>
+			<inertia
+			  ixx="5.6250000000000005e-05" ixy="0" ixz="0"
+			  iyy="5.6250000000000005e-05" iyz="0"
+			  izz="5.6250000000000005e-05"
 			/>
 		</inertial>
@@ -70,21 +70,20 @@
 			<origin xyz="0.0 0 0" rpy="0 1.5707 1.5707"/>
 			<geometry>
-				<cylinder radius="0.15" length="0.1"/>
-			</geometry>
-		</visual>
-		<collision name='collision'>
-			<origin xyz="0.0 0 0" rpy="0 1.5707 1.5707"/>
-			<geometry>
-				<cylinder radius="0.15" length="0.1"/>
-			</geometry>
-		</collision>
-		<inertial>
-			<mass value="10.0"/>
+				<cylinder radius="0.075" length="0.05"/>
+			</geometry>
+		</visual>
+		<collision name='collision'>
+			<origin xyz="0.0 0 0" rpy="0 1.5707 1.5707"/>
+			<geometry>
+				<cylinder radius="0.075" length="0.05"/>
+			</geometry>
+		</collision>
+		<inertial>
+			<mass value="1"/>
 			<origin xyz="0.0 0 0" rpy="0 1.5707 1.5707"/>
 				<inertia
-			  ixx="0.0646" ixy="0" ixz="0"
-			  iyy="0.0646" iyz="0"
-			  izz="0.1125"
-			/>
+			  ixx="0.0016145833333333329" ixy="0" ixz="0"
+			  iyy="0.0016145833333333329" iyz="0"
+			  izz="0.0028125"/>
 		</inertial>
 	</link>
@@ -94,20 +93,20 @@
 			<origin xyz="0.0 0 0" rpy="0 1.5707 1.5707"/>
 			<geometry>
-				<cylinder radius="0.15" length="0.1"/>
-			</geometry>
-		</visual>
-		<collision name='collision'>
-			<origin xyz="0.0 0 0" rpy="0 1.5707 1.5707"/>
-			<geometry>
-				<cylinder radius="0.15" length="0.1"/>
-			</geometry>
-		</collision>
-		<inertial>
-			<mass value="10.0"/>
+				<cylinder radius="0.075" length="0.05"/>
+			</geometry>
+		</visual>
+		<collision name='collision'>
+			<origin xyz="0.0 0 0" rpy="0 1.5707 1.5707"/>
+			<geometry>
+				<cylinder radius="0.075" length="0.05"/>
+			</geometry>
+		</collision>
+		<inertial>
+			<mass value="1"/>
 			<origin xyz="0.0 0 0" rpy="0 1.5707 1.5707"/>
 				<inertia
-			  ixx="0.0646" ixy="0" ixz="0"
-			  iyy="0.0646" iyz="0"
-			  izz="0.1125"/>
+			  ixx="0.0016145833333333329" ixy="0" ixz="0"
+			  iyy="0.0016145833333333329" iyz="0"
+			  izz="0.0028125"/>
 		</inertial>
 	</link>
@@ -116,10 +115,10 @@
 		<visual>
 		  <geometry>
-				<cylinder length="0.8" radius="0.1"/>
+				<cylinder length="0.4" radius="0.05"/>
 		  </geometry>
 		</visual>
 		<collision name='body_collision'>
 		  <geometry>
-				<cylinder length="0.65" radius="0.1"/>
+				<cylinder length="0.4" radius="0.05"/>
 		  </geometry>
 		</collision>
@@ -127,7 +126,7 @@
 			<mass value="0.1"/>
 			<inertia
-			  ixx="0.00558" ixy="0" ixz="0"
-			  iyy="0.00558" iyz="0"
-			  izz="0.00050"
+			  ixx="8.333333333333334e-05" ixy="0" ixz="0"
+			  iyy="8.333333333333334e-05" iyz="0"
+			  izz="0.00012500000000000003"
 			/>
 		</inertial>
@@ -137,10 +136,10 @@
 		<visual>
 			<geometry>
-				<box size="0.025 0.25 0.025"/>
-			</geometry>
-		</visual>
-		<collision name='collision'>
-			<geometry>
-				<box size="0.025 0.25 0.025"/>
+				<box size="0.0125 0.125 0.0125"/>
+			</geometry>
+		</visual>
+		<collision name='collision'>
+			<geometry>
+				<box size="0.0125 0.125 0.0125"/>
 			</geometry>
 		</collision>
@@ -165,12 +164,10 @@
 		</visual>
 		<collision name='collision'>
-			<origin xyz="0.0 0 0" rpy="0 0 0"/>
-			<geometry>
-				<box size="0.1 0.1 0.1"/>
+			<geometry>
+				<box size="0.05 0.05 0.05"/>
 			</geometry>
 		</collision>
 		<inertial>
 			<mass value="0.05"/>
-			<origin xyz="0.0 0 0" rpy="0 0 0"/>
 			<inertia
 			  ixx="1e-6" ixy="0" ixz="0"
@@ -182,5 +179,5 @@
 	<!-- Joint Robot footprint  -->
   <joint name="robot_footprint_joint" type="fixed">
-	  <origin xyz="0 0 0.15" rpy="0 0 0" />
+	  <origin xyz="0 0 0.075" rpy="0 0 0" />
     <parent link="robot_footprint"/>
     <child link="chassis_link"/>
@@ -188,6 +185,12 @@
 	<!-- Joint left wheel  -->
 	<joint name="left_wheel_joint" type="continuous" >
-		<origin xyz="0 0.35 0" rpy="0 0 0"/>
-		<axis xyz="0 1 0" />
+		<origin xyz="0 0.175 0" rpy="0 0 0"/>
+		<axis xyz="0 1 0">
+			<dynamics>
+				<damping>1.0</damping>
+				<friction>1.0</friction>
+			</dynamics>
+		</axis>
+		<limit effort="10000" velocity="1000"/>
 		<parent link="chassis_link"/>
 		<child link="left_wheel_link"/>
@@ -195,6 +198,12 @@
 	<!-- Joint right wheel  -->
 	<joint name="right_wheel_joint" type="continuous" >
-    <origin xyz="0 -0.35 0" rpy="0 0 0"/>
-		<axis xyz="0 1 0" />
+    <origin xyz="0 -0.175 0" rpy="0 0 0"/>
+		<axis xyz="0 1 0">
+			<dynamics>
+				<damping>1.0</damping>
+				<friction>1.0</friction>
+			</dynamics>
+		</axis>
+		<limit effort="10000" velocity="1000"/>
 		<parent link="chassis_link"/>
 		<child link="right_wheel_link"/>
@@ -202,5 +211,5 @@
 	<!-- Joint front caster  -->
 	<joint name="front_caster_joint" type="fixed" >
-		<origin xyz="0.22 0 -0.075" rpy="0 0 0"/>
+		<origin xyz="0.11 0 -0.0375" rpy="0 0 0"/>
 		<parent link="chassis_link"/>
 		<child link="front_caster_link"/>
@@ -208,5 +217,5 @@
 	<!-- Joint back caster  -->
 	<joint name="back_caster_joint" type="fixed" >
-		<origin xyz="-0.22 0 -0.075" rpy="0 0 0"/>
+		<origin xyz="-0.11 0 -0.0375" rpy="0 0 0"/>
 		<parent link="chassis_link"/>
 		<child link="back_caster_link"/>
@@ -214,5 +223,5 @@
 	<!-- Joint body  -->
 	<joint name="body_joint" type="fixed" >
-		<origin xyz="0 0 0.45" rpy="0 0 0"/>
+		<origin xyz="-0.015 0 0.225" rpy="0 0 0"/>
 		<parent link="chassis_link"/>
 		<child link="body_link"/>
@@ -220,5 +229,5 @@
 	<!-- Joint lidar  -->
 	<joint name="lidar_joint" type="fixed" >
-    <origin xyz="0 0 0.435" rpy="0 0 0"/>
+    <origin xyz="0 0 0.2175" rpy="0 0 0"/>
 		<parent link="body_link"/>
 		<child link="hokuyo"/>
@@ -226,5 +235,5 @@
 	<!-- Joint camera  -->
 	<joint name="camera_joint" type="fixed" >
-    <origin xyz="0.11 0 0.2" rpy="0 0 0"/>
+    <origin xyz="0.055 0 0.1" rpy="0 0 0"/>
 		<parent link="body_link"/>
 		<child link="camera_link"/>
